File: pcb/barracuda/barracuda.kicad_pcb (KiCad board)
At the start: 2 copper layers, 69 parts, among them SW1 SW_PUSH, SW10 SW_PUSH, SW11 SW_PUSH, SW12 SW_PUSH, SW13 SW_PUSH, SW14 SW_PUSH, SW15 SW_PUSH, SW16 SW_PUSH, SW17 SW_PUSH, SW18 SW_PUSH, SW19 SW_PUSH, SW2 SW_PUSH, SW20 SW_PUSH, SW21 SW_PUSH, SW22 SW_PUSH, SW23 SW_PUSH, SW24 SW_PUSH, SW25 SW_PUSH, SW26 SW_PUSH, SW27 SW_PUSH, SW28 SW_PUSH, SW29 SW_PUSH, SW3 SW_PUSH, SW30 SW_PUSH, SW31 SW_PUSH, SW32 SW_PUSH, SW33 SW_PUSH, SW4 SW_PUSH, SW5 SW_PUSH, SW6 SW_PUSH, SW7 SW_PUSH, SW8 SW_PUSH, SW9 SW_PUSH, U1 ProMicro

Commit message: Determined keyswitch layout and footprint
Parts:
- moved SW33 260.8 mm to (297.6, 88.1)
- moved SW30 243.1 mm to (278.6, 88.1)
- moved SW25 238.9 mm to (259.6, 50.0)
- moved SW32 237.7 mm to (297.6, 69.0)
- moved SW27 223.7 mm to (259.6, 88.1)
- moved SW29 220.0 mm to (278.6, 69.0)
- moved SW31 201.8 mm to (297.6, 50.0)
- moved SW28 196.6 mm to (278.6, 50.0)
- moved SW26 188.1 mm to (259.6, 69.0)
- moved SW24 182.8 mm to (240.5, 88.1)
- moved SW20 176.6 mm to (221.4, 69.0)
- moved SW23 159.3 mm to (240.5, 69.0)
- moved SW19 153.8 mm to (221.4, 50.0)
- moved SW6 148.1 mm to (69.0, 88.1)
- moved SW22 135.8 mm to (240.5, 50.0)
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
Commit message: Located mounting holes
Parts:
- added HOLE1: , kbd:HOLE, F.Cu at (59.5, 59.5)
- added HOLE13: , kbd:HOLE, F.Cu at (135.7, 59.5)
- added HOLE14: , kbd:HOLE, F.Cu at (135.7, 78.6)
- added HOLE2: , kbd:HOLE, F.Cu at (59.5, 78.6)
- added HOLE22: , kbd:HOLE, F.Cu at (250.0, 59.5)
- added HOLE23: , kbd:HOLE, F.Cu at (250.0, 78.6)
- added HOLE28: , kbd:HOLE, F.Cu at (288.1, 59.5)
- added HOLE29: , kbd:HOLE, F.Cu at (288.1, 78.6)
- added HOLE7: , kbd:HOLE, F.Cu at (97.6, 59.5)
- added HOLE8: , kbd:HOLE, F.Cu at (97.6, 78.6)
- moved LED1 13.9 mm to (29.5, 137.5)
- moved RSTSW1 12.7 mm to (37.0, 137.4)
Changed lines of the file:
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@@
     (tracks 0)
     (zones 0)
-    (modules 69)
+    (modules 79)
     (nets 57)
   )
@@
     (add_net row5)
   )
+  (module kbd:HOLE (layer F.Cu)
+    (at 288.125 78.575)
+    (descr "Mounting Hole 2.2mm, no annular, M2")
+    (tags "mounting hole 2.2mm no annular m2")
+    (attr virtual)
+    (fp_text reference HOLE29 (at 0 -3.2) (layer F.Fab)
+      (effects (font (size 1 1) (thickness 0.15)))
+    )
+    (fp_text value "" (at 0 3.2) (layer F.Fab)
+      (effects (font (size 1 1) (thickness 0.15)))
+    )
+    (fp_circle (center 0 0) (end 2.2 0) (layer Cmts.User) (width 0.15))
+    (fp_circle (center 0 0) (end 2.45 0) (layer F.CrtYd) (width 0.05))
+    (fp_text user %R (at 0.3 0) (layer F.Fab)
+      (effects (font (size 1 1) (thickness 0.15)))
+    )
+    (pad "" np_thru_hole circle (at 0 0) (size 5 5) (drill 4.8) (layers *.Cu *.Mask))
+  )
+  (module kbd:HOLE (layer F.Cu)
+    (at 288.125 59.525)
+    (descr "Mounting Hole 2.2mm, no annular, M2")
+    (tags "mounting hole 2.2mm no annular m2")
+    (attr virtual)
+    (fp_text reference HOLE28 (at 0 -3.2) (layer F.Fab)
+      (effects (font (size 1 1) (thickness 0.15)))
+    )
+    (fp_text value "" (at 0 3.2) (layer F.Fab)
+      (effects (font (size 1 1) (thickness 0.15)))
+    )
+    (fp_circle (center 0 0) (end 2.45 0) (layer F.CrtYd) (width 0.05))
+    (fp_circle (center 0 0) (end 2.2 0) (layer Cmts.User) (width 0.15))
+    (fp_text user %R (at 0.3 0) (layer F.Fab)
+      (effects (font (size 1 1) (thickness 0.15)))
+    )
+    (pad "" np_thru_hole circle (at 0 0) (size 5 5) (drill 4.8) (layers *.Cu *.Mask))
+  )
+  (module kbd:HOLE (layer F.Cu)
+    (at 250.025 78.575)
+    (descr "Mounting Hole 2.2mm, no annular, M2")
+    (tags "mounting hole 2.2mm no annular m2")
+    (attr virtual)
+    (fp_text reference HOLE23 (at 0 -3.2) (layer F.Fab)
+      (effects (font (size 1 1) (thickness 0.15)))
+    )
+    (fp_text value "" (at 0 3.2) (layer F.Fab)
+      (effects (font (size 1 1) (thickness 0.15)))
+    )
+    (fp_circle (center 0 0) (end 2.2 0) (layer Cmts.User) (width 0.15))
+    (fp_circle (center 0 0) (end 2.45 0) (layer F.CrtYd) (width 0.05))
+    (fp_text user %R (at 0.3 0) (layer F.Fab)
+      (effects (font (size 1 1) (thickness 0.15)))
+    )
+    (pad "" np_thru_hole circle (at 0 0) (size 5 5) (drill 4.8) (layers *.Cu *.Mask))
+  )
+  (module kbd:HOLE (layer F.Cu)
+    (at 250.025 59.525)
+    (descr "Mounting Hole 2.2mm, no annular, M2")
+    (tags "mounting hole 2.2mm no annular m2")
+    (attr virtual)
+    (fp_text reference HOLE22 (at 0 -3.2) (layer F.Fab)
+      (effects (font (size 1 1) (thickness 0.15)))
+    )
+    (fp_text value "" (at 0 3.2) (layer F.Fab)
+      (effects (font (size 1 1) (thickness 0.15)))
+    )
+    (fp_circle (center 0 0) (end 2.45 0) (layer F.CrtYd) (width 0.05))
+    (fp_circle (center 0 0) (end 2.2 0) (layer Cmts.User) (width 0.15))
+    (fp_text user %R (at 0.3 0) (layer F.Fab)
+      (effects (font (size 1 1) (thickness 0.15)))
+    )
+    (pad "" np_thru_hole circle (at 0 0) (size 5 5) (drill 4.8) (layers *.Cu *.Mask))
+  )
+  (module kbd:HOLE (layer F.Cu)
+    (at 135.725 78.575)
+    (descr "Mounting Hole 2.2mm, no annular, M2")
+    (tags "mounting hole 2.2mm no annular m2")
+    (attr virtual)
+    (fp_text reference HOLE14 (at 0 -3.2) (layer F.Fab)
+      (effects (font (size 1 1) (thickness 0.15)))
+    )
+    (fp_text value "" (at 0 3.2) (layer F.Fab)
+      (effects (font (size 1 1) (thickness 0.15)))
+    )
+    (fp_circle (center 0 0) (end 2.2 0) (layer Cmts.User) (width 0.15))
+    (fp_circle (center 0 0) (end 2.45 0) (layer F.CrtYd) (width 0.05))
+    (fp_text user %R (at 0.3 0) (layer F.Fab)
+      (effects (font (size 1 1) (thickness 0.15)))
+    )
+    (pad "" np_thru_hole circle (at 0 0) (size 5 5) (drill 4.8) (layers *.Cu *.Mask))
+  )
+  (module kbd:HOLE (layer F.Cu)
+    (at 135.725 59.525)
+    (descr "Mounting Hole 2.2mm, no annular, M2")
+    (tags "mounting hole 2.2mm no annular m2")
+    (attr virtual)
+    (fp_text reference HOLE13 (at 0 -3.2) (layer F.Fab)
+      (effects (font (size 1 1) (thickness 0.15)))
+    )
+    (fp_text value "" (at 0 3.2) (layer F.Fab)
+      (effects (font (size 1 1) (thickness 0.15)))
+    )
+    (fp_circle (center 0 0) (end 2.45 0) (layer F.CrtYd) (width 0.05))
+    (fp_circle (center 0 0) (end 2.2 0) (layer Cmts.User) (width 0.15))
+    (fp_text user %R (at 0.3 0) (layer F.Fab)
+      (effects (font (size 1 1) (thickness 0.15)))
+    )
+    (pad "" np_thru_hole circle (at 0 0) (size 5 5) (drill 4.8) (layers *.Cu *.Mask))
+  )
+  (module kbd:HOLE (layer F.Cu)
+    (at 97.625 78.575)
+    (descr "Mounting Hole 2.2mm, no annular, M2")
+    (tags "mounting hole 2.2mm no annular m2")
+    (attr virtual)
+    (fp_text reference HOLE8 (at 0 -3.2) (layer F.Fab)
+      (effects (font (size 1 1) (thickness 0.15)))
+    )
+    (fp_text value "" (at 0 3.2) (layer F.Fab)
+      (effects (font (size 1 1) (thickness 0.15)))
+    )
+    (fp_circle (center 0 0) (end 2.2 0) (layer Cmts.User) (width 0.15))
+    (fp_circle (center 0 0) (end 2.45 0) (layer F.CrtYd) (width 0.05))
+    (fp_text user %R (at 0.3 0) (layer F.Fab)
+      (effects (font (size 1 1) (thickness 0.15)))
+    )
+    (pad "" np_thru_hole circle (at 0 0) (size 5 5) (drill 4.8) (layers *.Cu *.Mask))
+  )
+  (module kbd:HOLE (layer F.Cu)
+    (at 97.625 59.525)
+    (descr "Mounting Hole 2.2mm, no annular, M2")
+    (tags "mounting hole 2.2mm no annular m2")
+    (attr virtual)
+    (fp_text reference HOLE7 (at 0 -3.2) (layer F.Fab)
+      (effects (font (size 1 1) (thickness 0.15)))
+    )
+    (fp_text value "" (at 0 3.2) (layer F.Fab)
+      (effects (font (size 1 1) (thickness 0.15)))
+    )
+    (fp_circle (center 0 0) (end 2.45 0) (layer F.CrtYd) (width 0.05))
+    (fp_circle (center 0 0) (end 2.2 0) (layer Cmts.User) (width 0.15))
+    (fp_text user %R (at 0.3 0) (layer F.Fab)
+      (effects (font (size 1 1) (thickness 0.15)))
+    )
+    (pad "" np_thru_hole circle (at 0 0) (size 5 5) (drill 4.8) (layers *.Cu *.Mask))
+  )
+  (module kbd:HOLE (layer F.Cu)
+    (at 59.525 78.575)
+    (descr "Mounting Hole 2.2mm, no annular, M2")
+    (tags "mounting hole 2.2mm no annular m2")
+    (attr virtual)
+    (fp_text reference HOLE2 (at 0 -3.2) (layer F.Fab)
+      (effects (font (size 1 1) (thickness 0.15)))
+    )
+    (fp_text value "" (at 0 3.2) (layer F.Fab)
+      (effects (font (size 1 1) (thickness 0.15)))
+    )
+    (fp_circle (center 0 0) (end 2.2 0) (layer Cmts.User) (width 0.15))
+    (fp_circle (center 0 0) (end 2.45 0) (layer F.CrtYd) (width 0.05))
+    (fp_text user %R (at 0.3 0) (layer F.Fab)
+      (effects (font (size 1 1) (thickness 0.15)))
+    )
+    (pad "" np_thru_hole circle (at 0 0) (size 5 5) (drill 4.8) (layers *.Cu *.Mask))
+  )
+  (module kbd:HOLE (layer F.Cu)
+    (at 59.525 59.525)
+    (descr "Mounting Hole 2.2mm, no annular, M2")
+    (tags "mounting hole 2.2mm no annular m2")
+    (attr virtual)
+    (fp_text reference HOLE1 (at 0 -3.2) (layer F.Fab)
+      (effects (font (size 1 1) (thickness 0.15)))
+    )
+    (fp_text value "" (at 0 3.2) (layer F.Fab)
+      (effects (font (size 1 1) (thickness 0.15)))
+    )
+    (fp_circle (center 0 0) (end 2.45 0) (layer F.CrtYd) (width 0.05))
+    (fp_circle (center 0 0) (end 2.2 0) (layer Cmts.User) (width 0.15))
+    (fp_text user %R (at 0.3 0) (layer F.Fab)
+      (effects (font (size 1 1) (thickness 0.15)))
+    )
+    (pad "" np_thru_hole circle (at 0 0) (size 5 5) (drill 4.8) (layers *.Cu *.Mask))
+  )
   (module kbd:D3_SMD (layer F.Cu)
     (at 41.656001 156.085001)
@@
   )
   (module LED_SMD:LED_WS2812B_PLCC4_5.0x5.0mm_P3.2mm (layer F.Cu)
-    (at 29.491001 151.400001)
+    (at 29.464 137.541)
     (descr https://cdn-shop.adafruit.com/datasheets/WS2812B.pdf)
     (tags "LED RGB NeoPixel")
@@
   )
   (module TVAF06-A020B-R:TVAF06-A020B-R (layer F.Cu)
-    (at 37.001 150.100001)
+    (at 36.957 137.414)
     (attr smd)
     (fp_text reference RSTSW1 (at 0 0.5) (layer F.SilkS)

Commit message: Located diodes (NOTE: some diodes conflict with mounting holes)
Parts:
- moved D31 298.1 mm to (303.9, 41.8), turned to 180 degrees
- moved D32 282.5 mm to (303.9, 60.8), turned to 180 degrees
- moved D28 275.8 mm to (284.9, 41.8), turned to 180 degrees
- moved D29 274.4 mm to (284.9, 60.8), turned to 180 degrees
- moved D33 269.5 mm to (303.9, 79.9), turned to 180 degrees
- moved D30 261.1 mm to (284.9, 79.9), turned to 180 degrees
- moved D25 245.8 mm to (265.8, 41.8), turned to 180 degrees
- moved D27 234.1 mm to (265.8, 79.9), turned to 180 degrees
- moved D22 220.4 mm to (246.8, 41.8), turned to 180 degrees
- moved D24 219.7 mm to (246.8, 79.9), turned to 180 degrees
- moved D23 217.3 mm to (246.8, 60.8), turned to 180 degrees
- moved D26 214.1 mm to (265.8, 60.8)
- moved D19 201.9 mm to (227.7, 41.8), turned to 180 degrees
- moved D20 197.4 mm to (227.7, 60.8), turned to 180 degrees
- moved D21 180.2 mm to (227.7, 79.9), turned to 180 degrees
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
Commit message: Resolved conflict of mounting holes and some diodes
Parts:
- moved D14 2.50 mm to (130.0, 60.8)
- moved D15 2.50 mm to (130.0, 79.9)
- moved D2 2.50 mm to (53.8, 60.8)
- moved D23 2.50 mm to (244.3, 60.8)
- moved D24 2.50 mm to (244.3, 79.9)
- moved D29 2.50 mm to (282.4, 60.8)
- moved D3 2.50 mm to (53.8, 79.9)
- moved D30 2.50 mm to (282.4, 79.9)
- moved D8 2.50 mm to (91.9, 60.8)
- moved D9 2.50 mm to (91.9, 79.9)

Commit message: Rough sketch of Edge.cuts
Parts:
- added HOLE21: , kbd:HOLE, F.Cu at (97.0, 35.4)
- added HOLE21: , kbd:HOLE, F.Cu at (83.7, 16.5)
- added HOLE21: , kbd:HOLE, F.Cu at (42.0, 16.5)
- added HOLE21: , kbd:HOLE, F.Cu at (42.0, 35.4)
- moved RSTSW1 123.5 mm to (83.3, 23.0)
- moved LED1 118.2 mm to (84.5, 32.9)
- moved U1 26.4 mm to (63.5, 26.9)
Other:
- board outline added: 271.4 x 87.6 mm
Changed lines of the file:
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@@
   (general
     (thickness 1.6)
-    (drawings 0)
+    (drawings 10)
     (tracks 0)
     (zones 0)
-    (modules 79)
+    (modules 83)
     (nets 57)
   )
@@
   )
   (module kbd:HOLE (layer F.Cu)
+    (at 97.028 35.433)
+    (descr "Mounting Hole 2.2mm, no annular, M2")
+    (tags "mounting hole 2.2mm no annular m2")
+    (attr virtual)
+    (fp_text reference HOLE21 (at 0 -3.2) (layer F.Fab)
+      (effects (font (size 1 1) (thickness 0.15)))
+    )
+    (fp_text value "" (at 0 3.2) (layer F.Fab)
+      (effects (font (size 1 1) (thickness 0.15)))
+    )
+    (fp_circle (center 0 0) (end 2.2 0) (layer Cmts.User) (width 0.15))
+    (fp_circle (center 0 0) (end 2.45 0) (layer F.CrtYd) (width 0.05))
+    (fp_text user %R (at 0.3 0) (layer F.Fab)
+      (effects (font (size 1 1) (thickness 0.15)))
+    )
+    (pad "" np_thru_hole circle (at 0 0) (size 5 5) (drill 4.8) (layers *.Cu *.Mask))
+  )
+  (module kbd:HOLE (layer F.Cu)
+    (at 83.693 16.51)
+    (descr "Mounting Hole 2.2mm, no annular, M2")
+    (tags "mounting hole 2.2mm no annular m2")
+    (attr virtual)
+    (fp_text reference HOLE21 (at 0 -3.2) (layer F.Fab)
+      (effects (font (size 1 1) (thickness 0.15)))
+    )
+    (fp_text value "" (at 0 3.2) (layer F.Fab)
+      (effects (font (size 1 1) (thickness 0.15)))
+    )
+    (fp_circle (center 0 0) (end 2.45 0) (layer F.CrtYd) (width 0.05))
+    (fp_circle (center 0 0) (end 2.2 0) (layer Cmts.User) (width 0.15))
+    (fp_text user %R (at 0.3 0) (layer F.Fab)
+      (effects (font (size 1 1) (thickness 0.15)))
+    )
+    (pad "" np_thru_hole circle (at 0 0) (size 5 5) (drill 4.8) (layers *.Cu *.Mask))
+  )
+  (module kbd:HOLE (layer F.Cu)
+    (at 42.037 16.51)
+    (descr "Mounting Hole 2.2mm, no annular, M2")
+    (tags "mounting hole 2.2mm no annular m2")
+    (attr virtual)
+    (fp_text reference HOLE21 (at 0 -3.2) (layer F.Fab)
+      (effects (font (size 1 1) (thickness 0.15)))
+    )
+    (fp_text value "" (at 0 3.2) (layer F.Fab)
+      (effects (font (size 1 1) (thickness 0.15)))
+    )
+    (fp_circle (center 0 0) (end 2.2 0) (layer Cmts.User) (width 0.15))
+    (fp_circle (center 0 0) (end 2.45 0) (layer F.CrtYd) (width 0.05))
+    (fp_text user %R (at 0.3 0) (layer F.Fab)
+      (effects (font (size 1 1) (thickness 0.15)))
+    )
+    (pad "" np_thru_hole circle (at 0 0) (size 5 5) (drill 4.8) (layers *.Cu *.Mask))
+  )
+  (module kbd:HOLE (layer F.Cu)
+    (at 42.037 35.433)
+    (descr "Mounting Hole 2.2mm, no annular, M2")
+    (tags "mounting hole 2.2mm no annular m2")
+    (attr virtual)
+    (fp_text reference HOLE21 (at 0 -3.2) (layer F.Fab)
+      (effects (font (size 1 1) (thickness 0.15)))
+    )
+    (fp_text value "" (at 0 3.2) (layer F.Fab)
+      (effects (font (size 1 1) (thickness 0.15)))
+    )
+    (fp_circle (center 0 0) (end 2.45 0) (layer F.CrtYd) (width 0.05))
+    (fp_circle (center 0 0) (end 2.2 0) (layer Cmts.User) (width 0.15))
+    (fp_text user %R (at 0.3 0) (layer F.Fab)
+      (effects (font (size 1 1) (thickness 0.15)))
+    )
+    (pad "" np_thru_hole circle (at 0 0) (size 5 5) (drill 4.8) (layers *.Cu *.Mask))
+  )
+  (module kbd:HOLE (layer F.Cu)
     (at 288.125 78.575)
     (descr "Mounting Hole 2.2mm, no annular, M2")
@@
   )
   (module LED_SMD:LED_WS2812B_PLCC4_5.0x5.0mm_P3.2mm (layer F.Cu)
-    (at 29.464 137.541)
+    (at 84.455 32.893)
     (descr https://cdn-shop.adafruit.com/datasheets/WS2812B.pdf)
     (tags "LED RGB NeoPixel")
@@
   )
   (module TVAF06-A020B-R:TVAF06-A020B-R (layer F.Cu)
-    (at 36.957 137.414)
+    (at 83.312 22.987)
     (attr smd)
     (fp_text reference RSTSW1 (at 0 0.5) (layer F.SilkS)
@@
   )
   (module Keebio-Parts:ArduinoProMicro (layer F.Cu)
-    (at 45.185001 45.910501)
+    (at 63.5 26.924)
     (fp_text reference U1 (at 0 1.625) (layer F.SilkS) hide
       (effects (font (size 1.27 1.524) (thickness 0.2032)))
@@
     )
   )
+  (gr_arc (start 41.91 16.51) (end 41.91 12.7) (angle -90) (layer Edge.Cuts) (width 0.05))
+  (gr_line (start 88.9 12.7) (end 41.91 12.7) (layer Edge.Cuts) (width 0.05))
+  (gr_line (start 114.3 38.1) (end 88.9 12.7) (layer Edge.Cuts) (width 0.05))
+  (gr_line (start 306.959 38.1) (end 114.3 38.1) (layer Edge.Cuts) (width 0.05))
+  (gr_arc (start 306.959 40.64) (end 309.499 40.64) (angle -90) (layer Edge.Cuts) (width 0.05))
+  (gr_line (start 309.499 97.79) (end 309.499 40.64) (layer Edge.Cuts) (width 0.05))
+  (gr_arc (start 306.959 97.79) (end 306.959 100.33) (angle -90) (layer Edge.Cuts) (width 0.05))
+  (gr_arc (start 40.64 97.79) (end 38.1 97.79) (angle -90) (layer Edge.Cuts) (width 0.05))
+  (gr_line (start 38.1 97.79) (end 38.1 16.51) (layer Edge.Cuts) (width 0.05))
+  (gr_line (start 40.64 100.33) (end 306.959 100.33) (layer Edge.Cuts) (width 0.05))
 )

Commit message: Created vias for all diodes
Parts:
- turned D26 to 180 degrees
Routing:
- net row2: track 0.00 -> 13.8 mm, vias 0 -> 6
- net row1: track 0.00 -> 13.8 mm, vias 0 -> 6
- net row0: track 0.00 -> 13.7 mm, vias 0 -> 6
- net row5: track 0.00 -> 11.5 mm, vias 0 -> 5
- net row4: track 0.00 -> 11.5 mm, vias 0 -> 5
- net row3: track 0.00 -> 11.4 mm, vias 0 -> 5
- net Net-(D2-Pad2): track 0.00 -> 2.83 mm, vias 0 -> 1
- net Net-(D9-Pad2): track 0.00 -> 2.58 mm, vias 0 -> 1
- net Net-(D8-Pad2): track 0.00 -> 2.58 mm, vias 0 -> 1
- net Net-(D30-Pad2): track 0.00 -> 2.58 mm, vias 0 -> 1
- net Net-(D29-Pad2): track 0.00 -> 2.58 mm, vias 0 -> 1
- net Net-(D23-Pad2): track 0.00 -> 2.58 mm, vias 0 -> 1
- net Net-(D3-Pad2): track 0.00 -> 2.58 mm, vias 0 -> 1
- net Net-(D14-Pad2): track 0.00 -> 2.58 mm, vias 0 -> 1
- net Net-(D24-Pad2): track 0.00 -> 2.32 mm, vias 0 -> 1
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
Commit message: Connected obvious tracks
Routing:
- net col4: track 0.00 -> 40.4 mm
- net col3: track 0.00 -> 40.4 mm
- net col0: track 0.00 -> 40.4 mm
- net col2: track 0.00 -> 40.4 mm
- net col1: track 0.00 -> 33.7 mm
- net Net-(D24-Pad2): track 2.32 -> 27.6 mm
- net Net-(D15-Pad2): track 2.32 -> 27.6 mm
- net Net-(D8-Pad2): track 2.58 -> 27.7 mm
- net Net-(D14-Pad2): track 2.58 -> 27.7 mm
- net Net-(D9-Pad2): track 2.58 -> 27.7 mm
- net Net-(D23-Pad2): track 2.58 -> 27.7 mm
- net Net-(D3-Pad2): track 2.58 -> 27.7 mm
- net Net-(D30-Pad2): track 2.58 -> 27.7 mm
- net Net-(D29-Pad2): track 2.58 -> 27.7 mm
- net Net-(D2-Pad2): track 2.83 -> 27.8 mm
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
Commit message: Connected trivial tracks
Parts:
- U1: moved to B.Cu
- moved U1 124.6 mm to (184.3, 57.5), turned to 270 degrees
Connections:
- D10 pad 1: row3 -> row0
- D11 pad 1: row4 -> row1
- D12 pad 1: row5 -> row2
- D16 pad 1: row3 -> row0
- D17 pad 1: row4 -> row1
- D18 pad 1: row5 -> row2
- D19 pad 1: row0 -> row3
- D20 pad 1: row1 -> row4
- D21 pad 1: row2 -> row5
- D25 pad 1: row0 -> row3
- D26 pad 1: row1 -> row4
- D27 pad 1: row2 -> row5
- D31 pad 1: row0 -> row3
- D32 pad 1: row1 -> row4
- D33 pad 1: row2 -> row5
- D4 pad 1: row3 -> row0
- D5 pad 1: row4 -> row1
- D6 pad 1: row5 -> row2
- SW10 pad 1: col1 -> col3
- SW11 pad 1: col1 -> col3
- SW12 pad 1: col1 -> col3
- SW13 pad 1: col2 -> col4
- SW14 pad 1: col2 -> col4
- SW15 pad 1: col2 -> col4
- SW16 pad 1: col2 -> col5
- SW17 pad 1: col2 -> col5
- SW18 pad 1: col2 -> col5
- SW19 pad 1: col3 -> col1
- SW20 pad 1: col3 -> col1
- SW21 pad 1: col3 -> col1
- SW22 pad 1: col3 -> col2
- SW23 pad 1: col3 -> col2
- SW24 pad 1: col3 -> col2
- SW25 pad 1: col4 -> col3
- SW26 pad 1: col4 -> col3
- SW27 pad 1: col4 -> col3
- SW4 pad 1: col0 -> col1
- SW5 pad 1: col0 -> col1
- SW6 pad 1: col0 -> col1
- SW7 pad 1: col1 -> col2
- SW8 pad 1: col1 -> col2
- SW9 pad 1: col1 -> col2
Routing:
- net col5: track 20.2 -> 70.7 mm, vias 0 -> 6
- net col1: track 33.7 -> 70.7 mm, vias 0 -> 6
- net col2: track 40.4 -> 70.7 mm, vias 0 -> 6
- net col4: track 40.4 -> 70.7 mm, vias 0 -> 6
- net col3: track 40.4 -> 64.0 mm, vias 0 -> 6
- net col0: track 40.4 -> 35.4 mm, vias 0 -> 3
