File: pcb/barracuda/barracuda.kicad_pcb (KiCad board)
At the start: 2 copper layers, 271.4 x 87.6 mm, 83 parts, among them SW1 SW_PUSH, SW10 SW_PUSH, SW11 SW_PUSH, SW12 SW_PUSH, SW13 SW_PUSH, SW14 SW_PUSH, SW15 SW_PUSH, SW16 SW_PUSH, SW17 SW_PUSH, SW18 SW_PUSH, SW19 SW_PUSH, SW2 SW_PUSH, SW20 SW_PUSH, SW21 SW_PUSH, SW22 SW_PUSH, SW23 SW_PUSH, SW24 SW_PUSH, SW25 SW_PUSH, SW26 SW_PUSH, SW27 SW_PUSH, SW28 SW_PUSH, SW29 SW_PUSH, SW3 SW_PUSH, SW30 SW_PUSH, SW31 SW_PUSH, SW32 SW_PUSH, SW33 SW_PUSH, SW4 SW_PUSH, SW5 SW_PUSH, SW6 SW_PUSH, SW7 SW_PUSH, SW8 SW_PUSH, SW9 SW_PUSH, U1 ProMicro

Commit message: Connected each columns
Routing:
- net col3: track 64.0 -> 119.7 mm
- net col5: track 70.7 -> 119.7 mm
- net col1: track 70.7 -> 117.3 mm
- net col4: track 70.7 -> 115.0 mm
- net col2: track 70.7 -> 115.0 mm
- net col0: track 35.4 -> 57.5 mm
- net Net-(D6-Pad2): track 25.2 -> 39.4 mm
- net Net-(D17-Pad2): track 25.2 -> 39.4 mm
- net Net-(D1-Pad2): track 25.2 -> 39.4 mm
- net Net-(D12-Pad2): track 25.2 -> 39.4 mm
- net Net-(D11-Pad2): track 25.2 -> 39.4 mm
- net Net-(D21-Pad2): track 25.2 -> 39.3 mm
- net Net-(D32-Pad2): track 25.2 -> 39.2 mm
- net Net-(D33-Pad2): track 25.2 -> 39.2 mm
- net Net-(D30-Pad2): track 27.7 -> 41.6 mm
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
Commit message: Connected trivial tracks
Routing:
- net col1: track 117.3 -> 239.8 mm, vias 6 -> 12
- net col2: track 115.0 -> 237.3 mm, vias 6 -> 12
- net col5: track 119.7 -> 241.9 mm, vias 6 -> 12
- net col3: track 119.7 -> 241.5 mm, vias 6 -> 12
- net col4: track 115.0 -> 236.8 mm, vias 6 -> 12
- net col0: track 57.5 -> 118.7 mm, vias 3 -> 6

Commit message: connected rows
Routing:
- net row1: track 13.8 -> 118.6 mm
- net row2: track 13.8 -> 118.6 mm
- net row0: track 13.7 -> 112.3 mm
- net row4: track 11.5 -> 92.9 mm
- net row5: track 11.5 -> 92.9 mm
- net row3: track 11.4 -> 90.3 mm
- net col2: track 237.3 -> 235.9 mm
- net col1: track 239.8 -> 238.4 mm
- net col0: track 118.7 -> 117.8 mm
- net col5: track 241.9 -> 242.5 mm

Commit message: PCB almost done
Parts:
- moved HOLE21 170.5 mm to (203.1, 91.4)
- moved HOLE21 141.8 mm to (162.7, 91.1)
- moved LED1 115.1 mm to (183.4, 91.7)
- moved HOLE21 106.4 mm to (203.2, 42.3)
- moved RSTSW1 88.7 mm to (169.9, 42.3), turned to 270 degrees
- moved HOLE21 81.8 mm to (161.4, 41.9)
- moved U1 0.89 mm to (183.4, 57.5)
Connections:
- U1 pad 10: row3 -> row0
- U1 pad 11: row4 -> row1
- U1 pad 12: row5 -> row2
- U1 pad 7: row0 -> row3
- U1 pad 8: row1 -> row4
- U1 pad 9: row2 -> row5
Routing:
- net col1: track 238.4 -> 441.4 mm, vias 12 -> 14
- net col2: track 235.9 -> 435.7 mm, vias 12 -> 14
- net col3: track 241.9 -> 435.6 mm, vias 12 -> 14
- net col4: track 236.4 -> 426.6 mm, vias 12 -> 14
- net col5: track 242.5 -> 415.2 mm, vias 12 -> 13
- net col0: track 117.8 -> 276.9 mm
- net GND: track 0.00 -> 74.1 mm
- net row0: track 112.3 -> 185.7 mm
- net row1: track 118.6 -> 173.7 mm
- net led: track 0.00 -> 48.7 mm
- net row3: track 90.3 -> 136.5 mm
- net row5: track 92.9 -> 138.0 mm
- net row2: track 118.6 -> 159.8 mm
- net VCC: track 0.00 -> 41.1 mm
- net row4: track 92.9 -> 132.2 mm
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- added copper zone on B.Cu, net GND
- added copper zone on F.Cu, net GND
Other:
- board size 271.4 x 87.6 mm -> 271.4 x 62.2 mm

Commit message: Replaced KeySwitch and diode footprints
Parts:
- removed LED1: WS2812B, LED_SMD:LED_WS2812B_PLCC4_5.0x5.0mm_P3.2mm
- D1, D10, D11, D12, D13, D14, D15, D16, D17, D18, D19, D2, D20, D21, D22, D23, D24, D25, D26, D27, D28, D29, D3, D30, D31, D32, D33, D4, D5, D6, D7, D8, D9: footprint kbd:D3_SMD -> barracuda:D3_SMD
- SW1, SW10, SW11, SW12, SW13, SW14, SW15, SW16, SW17, SW18, SW19, SW2, SW20, SW21, SW22, SW23, SW24, SW25, SW26, SW27, SW28, SW29, SW3, SW30, SW31, SW32, SW33, SW4, SW5, SW6, SW7, SW8, SW9: footprint kbd:CherryMX_Choc_Hotswap -> kbd:ChocV1_V2_Hotswap
- moved D3 8.33 mm to (58.3, 86.9), turned to 270 degrees
Connections:
- U1 pad 1: led -> Net-(U1-Pad1)
Routing:
- net col1: track 441.4 -> 78.9 mm, vias 14 -> 0
- net col2: track 435.7 -> 76.2 mm, vias 14 -> 0
- net col3: track 435.6 -> 81.5 mm, vias 14 -> 0
- net col4: track 426.6 -> 76.2 mm, vias 14 -> 0
- net col5: track 415.2 -> 81.5 mm, vias 13 -> 0
- net col0: track 276.9 -> 38.1 mm, vias 6 -> 0
- net row0: track 185.7 -> 0.00 mm, vias 6 -> 0
- net row1: track 173.7 -> 0.00 mm, vias 6 -> 0
- net row2: track 159.8 -> 0.89 mm, vias 6 -> 1
- net row5: track 138.0 -> 0.00 mm, vias 5 -> 0
- net row3: track 136.5 -> 0.00 mm, vias 5 -> 0
- net row4: track 132.2 -> 0.00 mm, vias 5 -> 0
- net GND: track 74.1 -> 0.00 mm
- net led: track 48.7 -> 0.00 mm
- net VCC: track 41.1 -> 0.00 mm
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
Commit message: Connected most of rows/columns
Parts:
- removed HOLE21 (x4): , kbd:HOLE
- moved U1 37.5 mm to (185.8, 20.1)
- moved D8 8.33 mm to (96.4, 67.8), turned to 270 degrees
- moved D9 8.33 mm to (96.4, 86.9), turned to 270 degrees
- moved D23 8.33 mm to (248.8, 67.8), turned to 270 degrees
- moved D24 8.33 mm to (248.8, 86.9), turned to 270 degrees
- moved D2 8.33 mm to (58.3, 67.8), turned to 270 degrees
- moved D14 8.33 mm to (134.5, 67.8), turned to 270 degrees
- moved D15 8.33 mm to (134.5, 86.9), turned to 270 degrees
- moved D29 8.33 mm to (286.9, 67.8), turned to 270 degrees
- moved D30 8.33 mm to (286.9, 86.9), turned to 270 degrees
- moved D19 7.27 mm to (229.7, 48.8), turned to 270 degrees
- moved D20 7.27 mm to (229.7, 67.8), turned to 270 degrees
- moved D21 7.27 mm to (229.7, 86.9), turned to 270 degrees
- moved D7 7.27 mm to (96.4, 48.8), turned to 270 degrees
- moved D25 7.27 mm to (267.8, 48.8), turned to 270 degrees
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Routing:
- net col2: track 76.2 -> 239.9 mm, vias 0 -> 2
- net col1: track 78.9 -> 239.9 mm, vias 0 -> 2
- net col4: track 76.2 -> 235.4 mm, vias 0 -> 2
- net col3: track 81.5 -> 239.7 mm, vias 0 -> 2
- net col5: track 81.5 -> 235.3 mm, vias 0 -> 2
- net row1: track 0.00 -> 95.3 mm, vias 0 -> 10
- net row0: track 0.00 -> 95.3 mm, vias 0 -> 10
- net row2: track 0.89 -> 95.3 mm, vias 1 -> 10
- net row5: track 0.00 -> 76.2 mm, vias 0 -> 8
- net row4: track 0.00 -> 76.2 mm, vias 0 -> 8
- net row3: track 0.00 -> 76.2 mm, vias 0 -> 8
- net Net-(D9-Pad2): track 14.7 -> 7.43 mm
- net Net-(D8-Pad2): track 14.7 -> 7.43 mm
- net Net-(D23-Pad2): track 14.7 -> 7.43 mm
- net Net-(D24-Pad2): track 14.7 -> 7.43 mm
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Other:
- board size 271.4 x 62.2 mm -> 269 x 59.7 mm

Commit message: Updated the MCU to atmega32u2
Parts:
- added C1: 22p, Capacitor_SMD:C_0603_1608Metric_Pad1.08x0.95mm_HandSolder, B.Cu at (193.2, 62.5)
- added C2: 22p, Capacitor_SMD:C_0603_1608Metric_Pad1.08x0.95mm_HandSolder, B.Cu at (193.2, 71.8)
- added C3: 0.1u, Capacitor_SMD:C_0603_1608Metric_Pad1.08x0.95mm_HandSolder, B.Cu at (179.8, 60.2)
- added C4: 10u, Capacitor_SMD:C_0805_2012Metric_Pad1.18x1.45mm_HandSolder, B.Cu at (189.4, 59.9)
- added C5: 1u, Capacitor_SMD:C_0603_1608Metric_Pad1.08x0.95mm_HandSolder, B.Cu at (193.2, 59.7)
- added C6: 0.1u, Capacitor_SMD:C_0603_1608Metric_Pad1.08x0.95mm_HandSolder, B.Cu at (193.2, 74.5)
- added F1: Polyfuse_Small, barracuda:RESC1206X70N, B.Cu at (186.4, 50.4)
- added J1: USB_B_Micro, barracuda:HRS_ZX62R-B-5P, B.Cu at (183.5, 43.4)
- added R1: 22, Resistor_SMD:R_0805_2012Metric_Pad1.20x1.40mm_HandSolder, B.Cu at (182.1, 49.9)
- added R2: 22, Resistor_SMD:R_0805_2012Metric_Pad1.20x1.40mm_HandSolder, B.Cu at (184.2, 49.9)
- added R3: 10k, Resistor_SMD:R_0805_2012Metric_Pad1.20x1.40mm_HandSolder, B.Cu at (174.9, 65.7)
- added R4: 10k, Resistor_SMD:R_0805_2012Metric_Pad1.20x1.40mm_HandSolder, B.Cu at (174.9, 72.6)
- added Y1: Crystal_GND24_Small, Crystal:Crystal_SMD_SeikoEpson_FA238-4Pin_3.2x2.5mm_HandSoldering, B.Cu at (193.2, 67.2)
- RSTSW1: moved to B.Cu
- U1: value ProMicro -> ATmega32U2-AU; footprint Keebio-Parts:ArduinoProMicro -> Package_QFP:TQFP-32_7x7mm_P0.8mm
- moved U1 49.2 mm to (183.5, 69.2), turned to 180 degrees
- moved RSTSW1 3.74 mm to (173.6, 41.7), turned to 180 degrees
Connections:
- U1 pad 10: row0 -> Net-(U1-Pad10)
- U1 pad 11: row1 -> Net-(U1-Pad11)
- U1 pad 12: row2 -> Net-(U1-Pad12)
- U1 pad 14: Net-(U1-Pad14) -> col0
- U1 pad 15: col5 -> col1
- U1 pad 16: col4 -> col2
- U1 pad 18: col2 -> col4
- U1 pad 19: col1 -> Net-(U1-Pad19)
- U1 pad 20: col0 -> row3
- U1 pad 21: VCC -> row4
- U1 pad 22: reset -> Net-(U1-Pad22)
- U1 pad 23: GND -> row2
- U1 pad 24: Net-(U1-Pad24) -> reset
- U1 pad 4: GND -> VCC
- U1 pad 5: Net-(U1-Pad5) -> row5
- U1 pad 7: row3 -> Net-(U1-Pad7)
- U1 pad 8: row4 -> Net-(U1-Pad8)
- U1 pad 9: row5 -> col5
Routing:
- net VCC: track 0.00 -> 75.1 mm, vias 0 -> 2
- net GND: track 0.00 -> 59.4 mm
- net row0: track 95.3 -> 131.2 mm
- net row2: track 95.3 -> 128.4 mm
- net row1: track 95.3 -> 122.9 mm
- net d_p: track 0.00 -> 14.9 mm
- net d_m: track 0.00 -> 14.3 mm
- net Net-(C1-Pad1): track 0.00 -> 11.5 mm
- net Net-(C2-Pad1): track 0.00 -> 8.82 mm
- net Net-(C3-Pad1): track 0.00 -> 6.48 mm
- net reset: track 0.00 -> 4.49 mm
- net Net-(J1-Pad3): track 0.00 -> 3.47 mm
- net Net-(F1-Pad2): track 0.00 -> 3.45 mm
- net Net-(J1-Pad2): track 0.00 -> 2.81 mm
Other:
- outline, holes or cut-outs redrawn

Commit message: save
Connections:
- U1 pad 10: Net-(U1-Pad10) -> col0
- U1 pad 11: Net-(U1-Pad11) -> col1
- U1 pad 12: Net-(U1-Pad12) -> col2
- U1 pad 14: col0 -> col3
- U1 pad 15: col1 -> col4
- U1 pad 16: col2 -> col5
- U1 pad 17: col3 -> Net-(U1-Pad17)
- U1 pad 18: col4 -> Net-(U1-Pad18)
- U1 pad 9: col5 -> Net-(U1-Pad9)
Routing:
- net col2: track 239.9 -> 416.8 mm, vias 2 -> 4
- net col3: track 239.7 -> 416.3 mm, vias 2 -> 4
- net col1: track 239.9 -> 416.3 mm, vias 2 -> 4
- net col0: track 38.1 -> 205.7 mm, vias 0 -> 1
- net row0: track 131.2 -> 95.3 mm
- net row2: track 128.4 -> 95.3 mm
- net col5: track 235.3 -> 263.2 mm
- net row1: track 122.9 -> 95.3 mm
- net col4: track 235.4 -> 258.4 mm
- net Net-(R4-Pad1): track 0.00 -> 10.1 mm, vias 0 -> 2
- net GND: track 59.4 -> 61.6 mm, vias 0 -> 1
