File: pcb/barracuda/barracuda.kicad_pcb (KiCad board)
At the start: 2 copper layers, 269 x 59.7 mm, 91 parts, among them J1 USB_B_Micro, SW1 SW_PUSH, SW10 SW_PUSH, SW11 SW_PUSH, SW12 SW_PUSH, SW13 SW_PUSH, SW14 SW_PUSH, SW15 SW_PUSH, SW16 SW_PUSH, SW17 SW_PUSH, SW18 SW_PUSH, SW19 SW_PUSH, SW2 SW_PUSH, SW20 SW_PUSH, SW21 SW_PUSH, SW22 SW_PUSH, SW23 SW_PUSH, SW24 SW_PUSH, SW25 SW_PUSH, SW26 SW_PUSH, SW27 SW_PUSH, SW28 SW_PUSH, SW29 SW_PUSH, SW3 SW_PUSH, SW30 SW_PUSH, SW31 SW_PUSH, SW32 SW_PUSH, SW33 SW_PUSH, SW4 SW_PUSH, SW5 SW_PUSH, SW6 SW_PUSH, SW7 SW_PUSH, SW8 SW_PUSH, SW9 SW_PUSH, U1 ATmega32U2-AU, Y1 Crystal_GND24_Small

Commit message: Finished routing
Parts:
- moved J1 1.08 mm to (183.5, 42.4)
- moved RSTSW1 0.38 mm to (173.6, 42.0)
Connections:
- U1 pad 20: row3 -> Net-(U1-Pad20)
- U1 pad 21: row4 -> Net-(U1-Pad21)
- U1 pad 5: row5 -> Net-(U1-Pad5)
- U1 pad 7: Net-(U1-Pad7) -> row3
- U1 pad 8: Net-(U1-Pad8) -> row4
- U1 pad 9: Net-(U1-Pad9) -> row5
Routing:
- net col2: track 416.8 -> 263.5 mm, vias 4 -> 2
- net col3: track 416.3 -> 265.9 mm, vias 4 -> 2
- net col1: track 416.3 -> 265.9 mm, vias 4 -> 2
- net row3: track 76.2 -> 157.2 mm, vias 8 -> 10
- net row4: track 76.2 -> 140.4 mm, vias 8 -> 10
- net row5: track 76.2 -> 125.1 mm, vias 8 -> 10
- net row0: track 95.3 -> 140.1 mm, vias 10 -> 12
- net row2: track 95.3 -> 137.3 mm, vias 10 -> 12
- net reset: track 4.49 -> 32.2 mm
- net row1: track 95.3 -> 122.9 mm, vias 10 -> 12
- net col0: track 205.7 -> 198.2 mm, vias 1 -> 0
- net Net-(J1-Pad3): track 3.47 -> 4.55 mm
- net Net-(J1-Pad2): track 2.81 -> 3.89 mm
- net Net-(F1-Pad2): track 3.45 -> 4.53 mm
- net GND: track 61.6 -> 62.4 mm, vias 1 -> 2
Other:
- outline, holes or cut-outs redrawn

Commit message: Finalized routing
Parts:
- moved RSTSW1 1.47 mm to (175.1, 42.2)
Routing:
- net reset: track 32.2 -> 30.7 mm
Changed lines of the file:
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@@
     (thickness 1.6)
     (drawings 13)
-    (tracks 569)
+    (tracks 568)
     (zones 0)
     (modules 91)
@@
   )
   (setup
-    (last_trace_width 0.5)
+    (last_trace_width 0.25)
     (user_trace_width 0.5)
     (trace_clearance 0.2)
@@
   )
   (module TVAF06-A020B-R:TVAF06-A020B-R (layer B.Cu)
-    (at 173.609 42.037 180)
+    (at 175.0695 42.164 180)
     (attr smd)
     (fp_text reference RSTSW1 (at 0 -0.5 180) (layer B.SilkS)
@@
   (segment (start 175.123 66.415) (end 179.265 66.415) (width 0.25) (layer B.Cu) (net 42))
   (segment (start 174.879 66.659) (end 175.123 66.415) (width 0.25) (layer B.Cu) (net 42))
-  (segment (start 175.921502 46.699002) (end 171.359 42.1365) (width 0.25) (layer B.Cu) (net 42))
-  (segment (start 175.921502 66.316498) (end 175.921502 46.699002) (width 0.25) (layer B.Cu) (net 42))
-  (segment (start 171.359 42.1365) (end 171.359 41.656) (width 0.25) (layer B.Cu) (net 42))
-  (segment (start 175.579 66.659) (end 175.921502 66.316498) (width 0.25) (layer B.Cu) (net 42))
-  (segment (start 174.879 66.659) (end 175.579 66.659) (width 0.25) (layer B.Cu) (net 42))
+  (segment (start 175.90401 65.63399) (end 175.90401 47.628012) (width 0.25) (layer B.Cu) (net 42))
+  (segment (start 174.879 66.659) (end 175.90401 65.63399) (width 0.25) (layer B.Cu) (net 42))
+  (segment (start 172.8195 44.543502) (end 175.90401 47.628012) (width 0.25) (layer B.Cu) (net 42))
+  (segment (start 172.8195 42.164) (end 172.8195 44.543502) (width 0.25) (layer B.Cu) (net 42))
   (segment (start 41.7 91.8) (end 41.7 72.75) (width 0.25) (layer B.Cu) (net 43))
   (segment (start 41.7 72.75) (end 41.7 53.7) (width 0.25) (layer B.Cu) (net 43))

Commit message: Added credit
Other:
- board text added: "barracuda v1.0 by knaruo"
