File: pcb/barracuda/barracuda.sch (KiCad schematic (older format))
At the start: 79 parts, among them SW1 SW_PUSH, SW10 SW_PUSH, SW11 SW_PUSH, SW12 SW_PUSH, SW13 SW_PUSH, SW14 SW_PUSH, SW15 SW_PUSH, SW16 SW_PUSH, SW17 SW_PUSH, SW18 SW_PUSH, SW19 SW_PUSH, SW2 SW_PUSH, SW20 SW_PUSH, SW21 SW_PUSH, SW22 SW_PUSH, SW23 SW_PUSH, SW24 SW_PUSH, SW25 SW_PUSH, SW26 SW_PUSH, SW27 SW_PUSH, SW28 SW_PUSH, SW29 SW_PUSH, SW3 SW_PUSH, SW30 SW_PUSH, SW31 SW_PUSH, SW32 SW_PUSH, SW33 SW_PUSH, SW34 SW_PUSH, SW35 SW_PUSH, SW36 SW_PUSH, SW37 SW_PUSH, SW38 SW_PUSH, SW4 SW_PUSH, SW5 SW_PUSH, SW6 SW_PUSH, SW7 SW_PUSH, SW8 SW_PUSH, SW9 SW_PUSH, U1 ProMicro

Commit message: Issue8 barracuda lp (#9)
* Reduced to 33 keys

* Assigned footprint to each components

* Generated PCB from net list

* Determined keyswitch layout and footprint

* Located mounting holes

* Located diodes (NOTE: some diodes conflict with mounting holes)

* Resolved conflict of mounting holes and some diodes

* Rough sketch of Edge.cuts

* Created vias for all diodes

* Connected obvious tracks

* Reassigned col/rows

* Connected trivial tracks

* Connected each columns

* Connected trivial tracks

* connected rows

* PCB almost done

* Replaced KeySwitch and diode footprints

* Connected most of rows/columns

* Updated the MCU to atmega32u2

* save

* Finished routing

* Finalized routing

* Done with bottom plate

* Done with the top plate

* Added credit

* Generated gerber files

* Regenerated gerber files to avoid errors in JLCPCB
Parts:
- removed D34, D35, D36, D37, D38: D, symbol Device:D
- removed LED1: WS2812B, LED_SMD:LED_WS2812B_PLCC4_5.0x5.0mm_P3.2mm, symbol LED:WS2812B
- removed SW34, SW35, SW36, SW37, SW38: SW_PUSH, symbol kbd:SW_PUSH
- removed U1: ProMicro, symbol kbd:ProMicro
- added C1, C2: 22p, Capacitor_SMD:C_0603_1608Metric_Pad1.08x0.95mm_HandSolder, symbol Device:C_Small
- added C3: 0.1u, Capacitor_SMD:C_0603_1608Metric_Pad1.08x0.95mm_HandSolder, symbol Device:C
- added C4: 10u, Capacitor_SMD:C_0805_2012Metric_Pad1.18x1.45mm_HandSolder, symbol Device:C_Small
- added C5: 1u, Capacitor_SMD:C_0603_1608Metric_Pad1.08x0.95mm_HandSolder, symbol Device:C_Small
- added C6: 0.1u, Capacitor_SMD:C_0603_1608Metric_Pad1.08x0.95mm_HandSolder, symbol Device:C_Small
- added F1: Polyfuse_Small, barracuda:RESC1206X70N, symbol Device:Polyfuse_Small
- added J1: USB_B_Micro, barracuda:HRS_ZX62R-B-5P, symbol Connector:USB_B_Micro
- added R1, R2: 22, Resistor_SMD:R_0805_2012Metric_Pad1.20x1.40mm_HandSolder, symbol Device:R
- added R3: 10k, Resistor_SMD:R_0805_2012Metric_Pad1.20x1.40mm_HandSolder, symbol Device:R
- added R4: 10k, Resistor_SMD:R_0805_2012Metric_Pad1.20x1.40mm_HandSolder, symbol Device:R_Small
- added U1: ATmega32U2-AU, Package_QFP:TQFP-32_7x7mm_P0.8mm, symbol MCU_Microchip_ATmega:ATmega32U2-AU
- added Y1: Crystal_GND24_Small, Crystal:Crystal_SMD_SeikoEpson_FA238-4Pin_3.2x2.5mm_HandSoldering, symbol Device:Crystal_GND24_Small
- D1, D10, D11, D12, D13, D14, D15, D16, D17, D18, D19, D2, D20, D21, D22, D23, D24, D25, D26, D27, D28, D29, D3, D30, D31, D32, D33, D4, D5, D6, D7, D8, D9: footprint (none) -> barracuda:D3_SMD
- RSTSW1: footprint (none) -> TVAF06-A020B-R:TVAF06-A020B-R
- SW1, SW10, SW11, SW12, SW13, SW14, SW15, SW16, SW17, SW18, SW19, SW2, SW20, SW21, SW22, SW23, SW24, SW25, SW26, SW27, SW28, SW29, SW3, SW30, SW31, SW32, SW33, SW4, SW5, SW6, SW7, SW8, SW9: footprint (none) -> kbd:ChocV1_V2_Hotswap
Connections:
- net GND: now also C1.2, C2.2, C3.2, C4.2, C5.2, C6.2, J1.5 (GND), J1.6 (Shield), R4.2, U1.28 (UGND), U1.3 (GND), Y1.2, Y1.4
- net VCC: now also C4.1, C5.1, C6.1, F1.1, R3.1, U1.31 (UVCC), U1.32 (AVCC), U1.4 (VCC)
- net col0: now also U1.10 (PD4); no longer SW4.1, SW5.1, SW6.1
- net col1: now also SW19.1, SW20.1, SW21.1, SW4.1, SW5.1, SW6.1, U1.11 (PD5); no longer SW10.1, SW11.1, SW12.1, SW7.1, SW8.1, SW9.1
- net col2: now also SW22.1, SW23.1, SW24.1, SW7.1, SW8.1, SW9.1, U1.12 (PD6); no longer SW13.1, SW14.1, SW15.1, SW16.1, SW17.1, SW18.1
- net col3: now also SW10.1, SW11.1, SW12.1, SW25.1, SW26.1, SW27.1, U1.14 (PB0); no longer SW19.1, SW20.1, SW21.1, SW22.1, SW23.1, SW24.1
- net col4: now also SW13.1, SW14.1, SW15.1, U1.15 (PB1); no longer SW25.1, SW26.1, SW27.1
- net col5: now also SW16.1, SW17.1, SW18.1, U1.16 (PB2)
- net reset: now also R3.2, U1.24 (PC1/~RESET)
- net row0: now also D10.1 (K), D16.1 (K), D4.1 (K), U1.26 (PC4); no longer D19.1 (K), D25.1 (K), D31.1 (K)
- net row1: now also D11.1 (K), D17.1 (K), D5.1 (K), U1.25 (PC5); no longer D20.1 (K), D26.1 (K), D32.1 (K)
- net row2: now also D12.1 (K), D18.1 (K), D6.1 (K), U1.23 (PC6); no longer D21.1 (K), D27.1 (K), D33.1 (K)
- net row3: now also D19.1 (K), D25.1 (K), D31.1 (K), U1.7 (PD1); no longer D10.1 (K), D16.1 (K), D4.1 (K)
- net row4: now also D20.1 (K), D26.1 (K), D32.1 (K), U1.8 (PD2); no longer D11.1 (K), D17.1 (K), D5.1 (K)
- net row5: now also D21.1 (K), D27.1 (K), D33.1 (K), U1.9 (PD3); no longer D12.1 (K), D18.1 (K), D6.1 (K)
- new net: C1.1, U1.1 (XTAL1), Y1.1
- new net: R4.1, U1.13 (~HWB~/PD7)
- new net: C2.1, U1.2 (PC0/XTAL2), Y1.3
- new net: C3.1, U1.27 (UCAP)
- new net: F1.2, J1.1 (VBUS)
- new net: J1.2 (D-), R2.2
- new net: J1.3 (D+), R1.2
- new net d_m: R2.1, U1.30 (D-)
- new net d_p: R1.1, U1.29 (D+)
- no-connect marks 6 -> 9
Other:
- note removed: "LED"
- moved on the sheet: D10, D11, D12, D13, D14, D15, D16, D17, D18, D19, D20, D21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
